Commit message: 修改urdf模型

File: public/urdf/myRobot/urdf/robot.urdf (robot description, URDF)
Before this commit: robot robot, 13 links, 12 joints
Links:
- added link base_frameA_link
- added link base_frameB_link
Joints:
- added joint base_jointA: type fixed, parent base_link, child base_frameA_link, origin xyz=0.00000 0.00000 -1.3000 rpy=-3.14159 -0.00000 -1.74533
- added joint base_jointB: type fixed, parent base_link, child base_frameB_link, origin xyz=0.00000 0.00000 1.3000 rpy=0.00000 0.00000 -1.74533
- joint arm1-lower-arm_link_joint: axis -0.64380 -0.76499 -0.01767 -> -0.63144 -0.77543 0.00000; child arm1-lower-arm_link -> arm2-lower-arm_link; limit lower=-3.14000 upper=3.14000 effort=0.00000 velocity=0.00000 -> lower=-3.14000 upper=0.69778 effort=0.00000 velocity=0.00000; origin xyz=0.20740 0.24927 0.19751 rpy=0.00000 0.00000 0.00000 -> xyz=0.20984 0.25317 -0.18652 rpy=-0.00000 0.00000 -0.00000; parent arm1-wrist1_link -> arm2-wrist1_link
- joint arm1-tool_link_joint: axis 0.34994 0.93677 -0.00136 -> 0.36743 0.92929 0.03775; child arm1-tool_link -> arm2-tool_link; origin xyz=-0.02087 -0.27051 -0.10962 rpy=0.00000 0.00000 0.00000 -> xyz=-0.01782 -0.27490 0.10498 rpy=0.00000 0.00000 -0.00000; parent arm1-wrist3_link -> arm2-wrist3_link
- joint arm1-upper-arm_link_joint: axis 0.67366 -0.55817 0.48439 -> 0.68742 -0.54399 -0.48116; child arm1-upper-arm_link -> arm2-upper-arm_link; origin xyz=-0.31274 0.11475 -0.17261 rpy=0.00000 0.00000 0.00000 -> xyz=-0.32092 0.09888 0.17334 rpy=-0.00000 0.00000 0.00000; parent arm1-wrist2_link -> arm2-wrist2_link
- joint arm1-wrist1_link_joint: axis 0.00000 0.00000 1.00000 -> 0.01446 -0.00936 0.99985; child arm1-wrist1_link -> arm2-wrist1_link; origin xyz=-0.00610 -0.20361 1.72510 rpy=0.00000 0.00000 0.00000 -> xyz=0.01807 -0.14331 -1.71436 rpy=0.00000 0.00000 0.00000
- joint arm1-wrist2_link_joint: axis -0.64380 -0.76499 -0.01767 -> -0.63144 -0.77543 0.00000; child arm1-wrist2_link -> arm2-wrist2_link; limit lower=-3.14000 upper=3.14000 effort=0.00000 velocity=0.00000 -> lower=-1.04667 upper=4.18667 effort=0.00000 velocity=0.00000; origin xyz=-1.14014 0.65820 0.73462 rpy=0.00000 0.00000 0.00000 -> xyz=-1.12976 0.68237 -0.72754 rpy=0.00000 0.00000 0.00000; parent arm1-lower-arm_link -> arm2-lower-arm_link
- joint arm1-wrist3_link_joint: axis -0.46355 0.18542 0.86645 -> -0.45622 0.27878 -0.84507; child arm1-wrist3_link -> arm2-wrist3_link; limit lower=-3.14000 upper=3.14000 effort=0.00000 velocity=0.00000 -> lower=-6.28000 upper=6.28000 effort=0.00000 velocity=0.00000; origin xyz=-0.58191 0.50342 -0.54785 rpy=0.00000 0.00000 -0.00000 -> xyz=-0.58435 0.49341 0.55420 rpy=-0.00000 -0.00000 0.00000; parent arm1-upper-arm_link -> arm2-upper-arm_link
- joint arm2-lower-arm_link_joint: axis -0.63144 -0.77543 0.00000 -> -0.64380 -0.76499 -0.01767; child arm2-lower-arm_link -> arm1-lower-arm_link; limit lower=-3.14000 upper=3.14000 effort=0.00000 velocity=0.00000 -> lower=-3.14000 upper=0.69778 effort=0.00000 velocity=0.00000; origin xyz=0.20984 0.25317 -0.18652 rpy=-0.00000 0.00000 -0.00000 -> xyz=0.20740 0.24927 0.19751 rpy=0.00000 0.00000 0.00000; parent arm2-wrist1_link -> arm1-wrist1_link
- joint arm2-tool_link_joint: axis 0.36743 0.92929 0.03775 -> 0.34994 0.93677 -0.00136; child arm2-tool_link -> arm1-tool_link; origin xyz=-0.01782 -0.27490 0.10498 rpy=0.00000 0.00000 -0.00000 -> xyz=-0.02087 -0.27051 -0.10962 rpy=0.00000 0.00000 0.00000; parent arm2-wrist3_link -> arm1-wrist3_link
- joint arm2-upper-arm_link_joint: axis 0.68742 -0.54399 -0.48116 -> 0.67366 -0.55817 0.48439; child arm2-upper-arm_link -> arm1-upper-arm_link; origin xyz=-0.32092 0.09888 0.17334 rpy=-0.00000 0.00000 0.00000 -> xyz=-0.31274 0.11475 -0.17261 rpy=0.00000 0.00000 0.00000; parent arm2-wrist2_link -> arm1-wrist2_link
- joint arm2-wrist1_link_joint: axis 0.01446 -0.00936 0.99985 -> 0.00000 0.00000 1.00000; child arm2-wrist1_link -> arm1-wrist1_link; origin xyz=0.01807 -0.14331 -1.71436 rpy=0.00000 0.00000 0.00000 -> xyz=-0.00610 -0.20361 1.72510 rpy=0.00000 0.00000 0.00000
- joint arm2-wrist2_link_joint: axis -0.63144 -0.77543 0.00000 -> -0.64380 -0.76499 -0.01767; child arm2-wrist2_link -> arm1-wrist2_link; limit lower=-3.14000 upper=3.14000 effort=0.00000 velocity=0.00000 -> lower=-1.04667 upper=4.18667 effort=0.00000 velocity=0.00000; origin xyz=-1.12976 0.68237 -0.72754 rpy=0.00000 0.00000 0.00000 -> xyz=-1.14014 0.65820 0.73462 rpy=0.00000 0.00000 0.00000; parent arm2-lower-arm_link -> arm1-lower-arm_link
- joint arm2-wrist3_link_joint: axis -0.45622 0.27878 -0.84507 -> -0.46355 0.18542 0.86645; child arm2-wrist3_link -> arm1-wrist3_link; limit lower=-3.14000 upper=3.14000 effort=0.00000 velocity=0.00000 -> lower=-6.28000 upper=6.28000 effort=0.00000 velocity=0.00000; origin xyz=-0.58435 0.49341 0.55420 rpy=-0.00000 -0.00000 0.00000 -> xyz=-0.58191 0.50342 -0.54785 rpy=0.00000 0.00000 -0.00000; parent arm2-upper-arm_link -> arm1-upper-arm_link
